File: hardware/Snake_1d/Snake_1d.kicad_pcb (KiCad board)
At the start: 2 copper layers, 60 x 60 mm, 16 parts, among them J1 LED_strip_connector, J2 SPI, Q1 PMN48XP, SW1 SW_Push, U1 SN74LVC1G14DBV, U2 ATtiny85-20SU

Commit message: Fixes missing (silk) footprints
Parts:
- added Ref**: Val**, Amieiro:ground_FSilks, B.Cu at (147.6, 76.7)
- added Ref**: Val**, Amieiro:arrow_up_from_left, B.Cu at (150.0, 76.6)
- added Ref**: Val**, Amieiro:5v_FSilks, B.Cu at (156.0, 74.0)

Commit message: Moves kicad files to new (nightly) format
Other:
- net class Default removed

Commit message: Changes LED strip connector footprint to horizontal pin header
Parts:
- J1: footprint Connector_PinHeader_2.54mm:PinHeader_1x03_P2.54mm_Vertical -> Connector_PinHeader_2.54mm:PinHeader_1x03_P2.54mm_Horizontal
Changed lines of the file:
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@@
     )
   )
-  (footprint "Connector_PinHeader_2.54mm:PinHeader_1x03_P2.54mm_Vertical" (layer "F.Cu")
+  (footprint "Connector_PinHeader_2.54mm:PinHeader_1x03_P2.54mm_Horizontal" (layer "F.Cu")
     (at 147.475 74 90)
-    (descr "Through hole straight pin header, 1x03, 2.54mm pitch, single row")
-    (tags "Through hole pin header THT 1x03 2.54mm single row")
+    (descr "Through hole angled pin header, 1x03, 2.54mm pitch, 6mm pin length, single row")
+    (tags "Through hole angled pin header THT 1x03 2.54mm single row")
     (attr through_hole)
-    (fp_text reference "J1" (at 0 -2.33 90) (layer "F.SilkS") hide
+    (fp_text reference "J1" (at 4.385 -2.27 90) (layer "F.SilkS")
       (effects (font (size 1 1) (thickness 0.15)))
     )
-    (fp_text value "LED_strip_connector" (at 0 7.41 90) (layer "F.Fab")
+    (fp_text value "LED_strip_connector" (at 4.385 7.35 90) (layer "F.Fab")
       (effects (font (size 1 1) (thickness 0.15)))
     )
-    (fp_text user "${REFERENCE}" (at 0 2.54 180) (layer "F.Fab")
+    (fp_text user "${REFERENCE}" (at 2.77 2.54 180) (layer "F.Fab")
       (effects (font (size 1 1) (thickness 0.15)))
     )
+    (fp_line (start 1.042929 2.16) (end 1.44 2.16) (layer "F.SilkS") (width 0.12))
+    (fp_line (start 4.1 -0.08) (end 10.1 -0.08) (layer "F.SilkS") (width 0.12))
+    (fp_line (start 4.1 6.41) (end 4.1 -1.33) (layer "F.SilkS") (width 0.12))
+    (fp_line (start 1.11 -0.38) (end 1.44 -0.38) (layer "F.SilkS") (width 0.12))
+    (fp_line (start 4.1 0.28) (end 10.1 0.28) (layer "F.SilkS") (width 0.12))
+    (fp_line (start 1.44 3.81) (end 4.1 3.81) (layer "F.SilkS") (width 0.12))
+    (fp_line (start 10.1 5.46) (end 4.1 5.46) (layer "F.SilkS") (width 0.12))
+    (fp_line (start 1.44 1.27) (end 4.1 1.27) (layer "F.SilkS") (width 0.12))
+    (fp_line (start 4.1 -0.2) (end 10.1 -0.2) (layer "F.SilkS") (width 0.12))
+    (fp_line (start 4.1 -0.32) (end 10.1 -0.32) (layer "F.SilkS") (width 0.12))
+    (fp_line (start 4.1 0.16) (end 10.1 0.16) (layer "F.SilkS") (width 0.12))
+    (fp_line (start 1.042929 5.46) (end 1.44 5.46) (layer "F.SilkS") (width 0.12))
+    (fp_line (start 1.042929 4.7) (end 1.44 4.7) (layer "F.SilkS") (width 0.12))
+    (fp_line (start 10.1 2.92) (end 4.1 2.92) (layer "F.SilkS") (width 0.12))
+    (fp_line (start 1.44 -1.33) (end 1.44 6.41) (layer "F.SilkS") (width 0.12))
+    (fp_line (start -1.27 -1.27) (end 0 -1.27) (layer "F.SilkS") (width 0.12))
+    (fp_line (start 4.1 -1.33) (end 1.44 -1.33) (layer "F.SilkS") (width 0.12))
+    (fp_line (start 1.042929 2.92) (end 1.44 2.92) (layer "F.SilkS") (width 0.12))
+    (fp_line (start 10.1 0.38) (end 4.1 0.38) (layer "F.SilkS") (width 0.12))
+    (fp_line (start 4.1 2.16) (end 10.1 2.16) (layer "F.SilkS") (width 0.12))
+    (fp_line (start 10.1 4.7) (end 10.1 5.46) (layer "F.SilkS") (width 0.12))
+    (fp_line (start -1.27 0) (end -1.27 -1.27) (layer "F.SilkS") (width 0.12))
+    (fp_line (start 4.1 0.04) (end 10.1 0.04) (layer "F.SilkS") (width 0.12))
+    (fp_line (start 1.11 0.38) (end 1.44 0.38) (layer "F.SilkS") (width 0.12))
+    (fp_line (start 4.1 -0.38) (end 10.1 -0.38) (layer "F.SilkS") (width 0.12))
+    (fp_line (start 4.1 4.7) (end 10.1 4.7) (layer "F.SilkS") (width 0.12))
+    (fp_line (start 10.1 -0.38) (end 10.1 0.38) (layer "F.SilkS") (width 0.12))
+    (fp_line (start 10.1 2.16) (end 10.1 2.92) (layer "F.SilkS") (width 0.12))
+    (fp_line (start 1.44 6.41) (end 4.1 6.41) (layer "F.SilkS") (width 0.12))
+    (fp_line (start 10.55 -1.8) (end -1.8 -1.8) (layer "F.CrtYd") (width 0.05))
     (fp_line (start -1.8 -1.8) (end -1.8 6.85) (layer "F.CrtYd") (width 0.05))
-    (fp_line (start -1.8 6.85) (end 1.8 6.85) (layer "F.CrtYd") (width 0.05))
-    (fp_line (start 1.8 6.85) (end 1.8 -1.8) (layer "F.CrtYd") (width 0.05))
-    (fp_line (start 1.8 -1.8) (end -1.8 -1.8) (layer "F.CrtYd") (width 0.05))
-    (fp_line (start 1.27 6.35) (end -1.27 6.35) (layer "F.Fab") (width 0.1))
-    (fp_line (start -0.635 -1.27) (end 1.27 -1.27) (layer "F.Fab") (width 0.1))
-    (fp_line (start 1.27 -1.27) (end 1.27 6.35) (layer "F.Fab") (width 0.1))
-    (fp_line (start -1.27 -0.635) (end -0.635 -1.27) (layer "F.Fab") (width 0.1))
-    (fp_line (start -1.27 6.35) (end -1.27 -0.635) (layer "F.Fab") (width 0.1))
+    (fp_line (start -1.8 6.85) (end 10.55 6.85) (layer "F.CrtYd") (width 0.05))
+    (fp_line (start 10.55 6.85) (end 10.55 -1.8) (layer "F.CrtYd") (width 0.05))
+    (fp_line (start 4.04 -0.32) (end 10.04 -0.32) (layer "F.Fab") (width 0.1))
+    (fp_line (start -0.32 2.22) (end 1.5 2.22) (layer "F.Fab") (width 0.1))
+    (fp_line (start -0.32 5.4) (end 1.5 5.4) (layer "F.Fab") (width 0.1))
+    (fp_line (start 10.04 -0.32) (end 10.04 0.32) (layer "F.Fab") (width 0.1))
+    (fp_line (start -0.32 2.86) (end 1.5 2.86) (layer "F.Fab") (width 0.1))
+    (fp_line (start 2.135 -1.27) (end 4.04 -1.27) (layer "F.Fab") (width 0.1))
+    (fp_line (start 4.04 2.86) (end 10.04 2.86) (layer "F.Fab") (width 0.1))
+    (fp_line (start 4.04 4.76) (end 10.04 4.76) (layer "F.Fab") (width 0.1))
+    (fp_line (start 4.04 0.32) (end 10.04 0.32) (layer "F.Fab") (width 0.1))
+    (fp_line (start -0.32 4.76) (end -0.32 5.4) (layer "F.Fab") (width 0.1))
+    (fp_line (start 1.5 -0.635) (end 2.135 -1.27) (layer "F.Fab") (width 0.1))
+    (fp_line (start -0.32 -0.32) (end 1.5 -0.32) (layer "F.Fab") (width 0.1))
+    (fp_line (start 4.04 -1.27) (end 4.04 6.35) (layer "F.Fab") (width 0.1))
+    (fp_line (start 10.04 4.76) (end 10.04 5.4) (layer "F.Fab") (width 0.1))
+    (fp_line (start 4.04 5.4) (end 10.04 5.4) (layer "F.Fab") (width 0.1))
+    (fp_line (start -0.32 0.32) (end 1.5 0.32) (layer "F.Fab") (width 0.1))
+    (fp_line (start -0.32 -0.32) (end -0.32 0.32) (layer "F.Fab") (width 0.1))
+    (fp_line (start 4.04 6.35) (end 1.5 6.35) (layer "F.Fab") (width 0.1))
+    (fp_line (start 1.5 6.35) (end 1.5 -0.635) (layer "F.Fab") (width 0.1))
+    (fp_line (start 10.04 2.22) (end 10.04 2.86) (layer "F.Fab") (width 0.1))
+    (fp_line (start -0.32 4.76) (end 1.5 4.76) (layer "F.Fab") (width 0.1))
+    (fp_line (start 4.04 2.22) (end 10.04 2.22) (layer "F.Fab") (width 0.1))
+    (fp_line (start -0.32 2.22) (end -0.32 2.86) (layer "F.Fab") (width 0.1))
     (pad "1" thru_hole rect (at 0 0 90) (locked) (size 1.7 1.7) (drill 1) (layers *.Cu *.Mask)
       (net 1 "GND"))
@@
     (pad "3" thru_hole oval (at 0 5.08 90) (locked) (size 1.7 1.7) (drill 1) (layers *.Cu *.Mask)
       (net 5 "+5V"))
-    (model "${KISYS3DMOD}/Connector_PinHeader_2.54mm.3dshapes/PinHeader_1x03_P2.54mm_Vertical.wrl"
+    (model "${KISYS3DMOD}/Connector_PinHeader_2.54mm.3dshapes/PinHeader_1x03_P2.54mm_Horizontal.wrl"
       (offset (xyz 0 0 0))
       (scale (xyz 1 1 1))
