File: hardware/Snake_1d/Snake_1d.kicad_sch (KiCad schematic)
At the start: 16 parts, among them J1 LED_strip_connector, J2 SPI, Q1 PMN48XP, SW1 SW_Push, U1 SN74LVC1G14DBV, U2 ATtiny85-20SU

Commit message: Changes LED strip connector footprint to horizontal pin header
Parts:
- J1: footprint Connector_PinHeader_2.54mm:PinHeader_1x03_P2.54mm_Vertical -> Connector_PinHeader_2.54mm:PinHeader_1x03_P2.54mm_Horizontal
Changed lines of the file:
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@@
       (effects (font (size 1.27 1.27)) (justify right))
     )
-    (property "Footprint" "Connector_PinHeader_2.54mm:PinHeader_1x03_P2.54mm_Vertical" (id 2) (at 76.2 110.49 0)
+    (property "Footprint" "Connector_PinHeader_2.54mm:PinHeader_1x03_P2.54mm_Horizontal" (id 2) (at 76.2 110.49 0)
       (effects (font (size 1.27 1.27)) hide)
     )
@@
     )
     (path "/00000000-0000-0000-0000-00005f7faa68"
-      (reference "J1") (unit 1) (value "LED_strip_connector") (footprint "Connector_PinHeader_2.54mm:PinHeader_1x03_P2.54mm_Vertical")
+      (reference "J1") (unit 1) (value "LED_strip_connector") (footprint "Connector_PinHeader_2.54mm:PinHeader_1x03_P2.54mm_Horizontal")
     )
     (path "/00000000-0000-0000-0000-00005f806264"
